Commit message: All encoders named 1,2,3,4

File: src/IRAC/urdf/irac.xacro (robot description, xacro)
@@ -18,5 +18,5 @@
   <!-- Used for fixing robot to Gazebo 'base_link' -->
   <link name="world"/>
-  <joint name="joint0" type="continuous">
+  <joint name="joint1" type="continuous">
     <parent link="world"/>
     <child link="link1"/>
@@ -49,5 +49,5 @@
     </inertial>
   </link>
-  <joint name="joint1" type="continuous">
+  <joint name="joint2" type="continuous">
     <parent link="link1"/>
     <child link="link2"/>
@@ -80,5 +80,5 @@
     </inertial>
   </link>
-  <joint name="joint2" type="continuous">
+  <joint name="joint3" type="continuous">
     <parent link="link2"/>
     <child link="link3"/>
@@ -111,5 +111,5 @@
     </inertial>
   </link>
-<joint name="joint3" type="continuous">
+<joint name="joint4" type="continuous">
     <parent link="link3"/>
     <child link="link4"/>
@@ -142,14 +142,4 @@
     </inertial>
   </link>
-  <transmission name="tran0">
-    <type>transmission_interface/SimpleTransmission</type>
-    <joint name="joint0">
-      <hardwareInterface>hardware_interface/EffortJointInterface</hardwareInterface>
-    </joint>
-    <actuator name="motor0">
-      <hardwareInterface>hardware_interface/EffortJointInterface</hardwareInterface>
-      <mechanicalReduction>1</mechanicalReduction>
-    </actuator>
-  </transmission>
   <transmission name="tran1">
     <type>transmission_interface/SimpleTransmission</type>
@@ -182,3 +172,13 @@
     </actuator>
   </transmission>
+  <transmission name="tran4">
+    <type>transmission_interface/SimpleTransmission</type>
+    <joint name="joint4">
+      <hardwareInterface>hardware_interface/EffortJointInterface</hardwareInterface>
+    </joint>
+    <actuator name="motor4">
+      <hardwareInterface>hardware_interface/EffortJointInterface</hardwareInterface>
+      <mechanicalReduction>1</mechanicalReduction>
+    </actuator>
+  </transmission>
 </robot>
