Commit message: IK solver returning values

File: src/sim_control/src/irac.urdf (robot description, URDF)
Before this commit: robot irac, 5 links, 4 joints
Links:
- added link flange
- link link1: mass None -> 0.4; geometry collision mesh filename=/home/kurt/Senior_Design/src/IRAC/urdf/meshes/Base.stl scale=.001 .001 .001; visual mesh filename=/home/kurt/Senior_Design/src/IRAC/urdf/meshes/Base.stl scale=.001 .001 .001
- link link2: mass None -> 0.4; geometry collision mesh filename=/home/kurt/Senior_Design/src/IRAC/urdf/meshes/Link1.stl scale=.001 .001 .001; visual mesh filename=/home/kurt/Senior_Design/src/IRAC/urdf/meshes/Link1.stl scale=.001 .001 .001
- link link3: mass None -> 0.4; geometry collision mesh filename=/home/kurt/Senior_Design/src/IRAC/urdf/meshes/Link2.stl scale=.001 .001 .001; visual mesh filename=/home/kurt/Senior_Design/src/IRAC/urdf/meshes/Link2.stl scale=.001 .001 .001
- link link4: mass None -> 0.4; geometry collision mesh filename=/home/kurt/Senior_Design/src/IRAC/urdf/meshes/Link3.stl scale=.001 .001 .001; visual mesh filename=/home/kurt/Senior_Design/src/IRAC/urdf/meshes/Link3.stl scale=.001 .001 .001
Joints:
- added joint flange: type fixed, parent link4, child flange, origin xyz= 0.0 0.0 0.1206 rpy=0.0 0.0 0.0
- joint joint2: origin xyz=0 0.1 0.45 rpy=0 0 0 -> xyz=0 -0.0301625 .127175 rpy=0 0 0
- joint joint3: origin xyz=0 0.1 0.9 rpy=0 0 0 -> xyz=0 0 .28076 rpy=0 0 0
- joint joint4: origin xyz=0 0.1 0.85 rpy=0 0 0 -> xyz=0 .05237 .25975 rpy=0 0 0

File: src/sim_control/src/irac_noGazebo.xacro (robot description, xacro)
@@ -4,16 +4,40 @@
   <!-- Constants for robot dimensions -->
   <xacro:property name="PI" value="3.1415926535897931"/>
-  <xacro:property name="mass" value="1" /> <!-- arbitrary value for mass -->
-  <xacro:property name="width" value="0.1" /> <!-- Square dimensions (widthxwidth) of beams -->
-  <xacro:property name="height1" value=".5" /> <!-- Link 1 -->
-  <xacro:property name="height2" value="1" /> <!-- Link 2 -->
-  <xacro:property name="height3" value="1" /> <!-- Link 3 -->
-  <xacro:property name="height4" value=".5" /> <!-- Link 0 -->
-  <xacro:property name="camera_link" value="0.05" /> <!-- Size of square 'camera' box -->
-  <xacro:property name="axel_offset" value="0.05" /> <!-- Space btw top of beam and the each joint -->
+  <xacro:property name="mass" value=".4" /> <!-- arbitrary value for mass -->
+  <xacro:property name="width" value="0.06" /> <!-- Square dimensions (widthxwidth) of beams -->
+  <xacro:property name="height1" value=".1397" /> <!-- Link 1 -->
+  <xacro:property name="height2" value="0.32476" /> <!-- Link 2 -->
+  <xacro:property name="height3" value="0.28416" /> <!-- Link 3 -->
+  <xacro:property name="height4" value="0.12065" /> <!-- Link 0 -->
+  <xacro:property name="axel_offset" value="${.060325/2}" />
   <!-- Import Rviz colors -->
   <xacro:include filename="$(find IRAC)/urdf/materials.xacro" />
   <!-- Used for fixing robot to Gazebo 'base_link' -->
   <link name="world"/>
+  <!-- Link 1 || BASE -->
+  <link name="link1">
+    <collision>
+      <origin xyz="0 0 0" rpy="0 0 0"/>
+      <geometry>
+	      <mesh filename="$(find IRAC)/urdf/meshes/Base.stl" scale=".001 .001 .001"/>
+      </geometry>
+    </collision>
+    <visual>
+      <origin xyz="0 0 0" rpy="0 0 0"/>
+      <geometry>
+	      <mesh filename="$(find IRAC)/urdf/meshes/Base.stl" scale=".001 .001 .001"/>
+      </geometry>
+      <material name="orange"/>
+    </visual>
+    <inertial>
+      <origin xyz="0 0 0" rpy="0 0 0"/>
+      <mass value="${mass}"/>
+      <inertia
+	      ixx="${mass / 12.0 * (width*width + height1*height1)}" ixy="0.0" ixz="0.0"
+	      iyy="${mass / 12.0 * (height1*height1 + width*width)}" iyz="0.0"
+	      izz="${mass / 12.0 * (width*width + width*width)}"/>
+    </inertial>
+  </link>
+  <!-- JOINT 1 -->
   <joint name="joint1" type="continuous">
     <parent link="world"/>
@@ -22,89 +46,110 @@
     <axis xyz="0 0 1"/>
     <dynamics damping="0.7"/>
-  </joint>
-  <!-- Base Link -->
-  <link name="link1">
-    <collision>
-      <origin xyz="0 0 ${height1/2}" rpy="0 0 0"/>
-      <geometry>
-	<box size="${width} ${width} ${height1}"/>
-      </geometry>
-    </collision>
-    <visual>
-      <origin xyz="0 0 ${height1/2}" rpy="0 0 0"/>
-      <geometry>
-	<box size="${width} ${width} ${height1}"/>
-      </geometry>
-      <material name="orange"/>
-    </visual>
-  </link>
-  <joint name="joint2" type="continuous">
-    <parent link="link1"/>
-    <child link="link2"/>
-    <origin xyz="0 ${width} ${height1 - axel_offset}" rpy="0 0 0"/>
-    <axis xyz="0 1 0"/>
-    <dynamics damping="0.7"/>
+    <!-- <limit lower="${-PI/2}" upper="${PI/2}" effort="30.0" velocity="10.0"/> -->
   </joint>
   <!-- Link 2 -->
   <link name="link2">
     <collision>
-      <origin xyz="0 0 ${height2/2 - axel_offset}" rpy="0 0 0"/>
+      <origin xyz="0 0 0" rpy="0 0 0"/>
       <geometry>
-	<box size="${width} ${width} ${height2}"/>
+	      <mesh filename="$(find IRAC)/urdf/meshes/Link1.stl" scale=".001 .001 .001"/>
       </geometry>
     </collision>
     <visual>
-      <origin xyz="0 0 ${height2/2 - axel_offset}" rpy="0 0 0"/>
+      <origin xyz="0 0 0" rpy="0 0 0"/>
       <geometry>
-	<box size="${width} ${width} ${height2}"/>
+	      <mesh filename="$(find IRAC)/urdf/meshes/Link1.stl" scale=".001 .001 .001"/>
       </geometry>
-      <material name="black"/>
+      <material name="blue"/>
     </visual>
+    <inertial>
+      <origin xyz="0 0 0" rpy="0 0 0"/>
+      <mass value="${mass}"/>
+      <inertia
+	      ixx="${mass / 12.0 * (width*width + height2*height2)}" ixy="0.0" ixz="0.0"
+	      iyy="${mass / 12.0 * (height2*height2 + width*width)}" iyz="0.0"
+	      izz="${mass / 12.0 * (width*width + width*width)}"/>
+    </inertial>
   </link>
+  <!-- JOINT 2 -->
+  <joint name="joint2" type="continuous">
+    <parent link="link1"/>
+    <child link="link2"/>
+    <origin xyz="0 ${-1*axel_offset} .127175" rpy="0 0 0"/>
+    <axis xyz="0 1 0"/>
+    <dynamics damping="0.7"/>
+    <!-- <limit lower="${-PI/2}" upper="${PI/2}" effort="30.0" velocity="10.0"/> -->
+  </joint>
+  <!-- Link 3 -->
+  <link name="link3">
+    <collision>
+      <origin xyz="0 0 0" rpy="0 0 0"/>
+      <geometry>
+	      <mesh filename="$(find IRAC)/urdf/meshes/Link2.stl" scale=".001 .001 .001"/>
+      </geometry>
+    </collision>
+    <visual>
+      <origin xyz="0 0 0" rpy="0 0 0"/>
+      <geometry>
+	      <mesh filename="$(find IRAC)/urdf/meshes/Link2.stl" scale=".001 .001 .001"/>
+      </geometry>
+      <material name="orange"/>
+    </visual>
+    <inertial>
+      <origin xyz="0 0 0" rpy="0 0 0"/>
+      <mass value="${mass}"/>
+      <inertia
+	      ixx="${mass / 12.0 * (width*width + height3*height3)}" ixy="0.0" ixz="0.0"
+	      iyy="${mass / 12.0 * (height3*height3 + width*width)}" iyz="0.0"
+	      izz="${mass / 12.0 * (width*width + width*width)}"/>
+    </inertial>
+  </link>
+  <!-- JOINT 3 -->
   <joint name="joint3" type="continuous">
     <parent link="link2"/>
     <child link="link3"/>
-    <origin xyz="0 ${width} ${height2 - axel_offset*2}" rpy="0 0 0"/>
+    <origin xyz="0 0 .28076" rpy="0 0 0"/>
     <axis xyz="0 1 0"/>
     <dynamics damping="0.7"/>
+    <!-- <limit lower="${-PI/2}" upper="${PI/2}" effort="30.0" velocity="10.0"/> -->
   </joint>
-  <!-- Top Link -->
-  <link name="link3">
+  <!-- LINK 4-->
+  <link name="link4">
     <collision>
-      <origin xyz="0 0 ${height3/2 - axel_offset}" rpy="0 0 0"/>
+      <origin xyz="0 0 0" rpy="0 0 0"/>
       <geometry>
-	<box size="${width} ${width} ${height3}"/>
+	      <mesh filename="$(find IRAC)/urdf/meshes/Link3.stl" scale=".001 .001 .001"/>
       </geometry>
     </collision>
     <visual>
-      <origin xyz="0 0 ${height3/2 - axel_offset}" rpy="0 0 0"/>
+      <origin xyz="0 0 0" rpy="0 0 0"/>
       <geometry>
-	<box size="${width} ${width} ${height3}"/>
+	      <mesh filename="$(find IRAC)/urdf/meshes/Link3.stl" scale=".001 .001 .001"/>
       </geometry>
       <material name="orange"/>
     </visual>
+    <inertial>
+      <origin xyz="0 0 0" rpy="0 0 0"/>
+      <mass value="${mass}"/>
+      <inertia
+	      ixx="${mass / 12.0 * (width*width + height4*height4)}" ixy="0.0" ixz="0.0"
+	      iyy="${mass / 12.0 * (height4*height4 + width*width)}" iyz="0.0"
+	      izz="${mass / 12.0 * (width*width + width*width)}"/>
+    </inertial>
   </link>
-<joint name="joint4" type="continuous">
+  <!-- JOINT 4 -->
+  <joint name="joint4" type="continuous">
     <parent link="link3"/>
     <child link="link4"/>
-    <origin xyz="0 ${width} ${height3 - axel_offset*3}" rpy="0 0 0"/>
+    <origin xyz="0 .05237 .25975" rpy="0 0 0"/>
     <axis xyz="0 1 0"/>
     <dynamics damping="0.7"/>
+    <!-- <limit lower="${-PI/2}" upper="${PI/2}" effort="30.0" velocity="10.0"/> -->
   </joint>
-  <!-- EAOT-->
-  <link name="link4">
-    <collision>
-      <origin xyz="0 0 ${height4/2 - axel_offset}" rpy="0 0 0"/>
-      <geometry>
-	<box size="${width} ${width} ${height4}"/>
-      </geometry>
-    </collision>
-    <visual>
-      <origin xyz="0 0 ${height4/2 - axel_offset}" rpy="0 0 0"/>
-      <geometry>
-	<box size="${width} ${width} ${height4}"/>
-      </geometry>
-      <material name="orange"/>
-    </visual>
-  </link>
+  <link name="flange"/>
+  <joint name="flange" type="fixed">
+    <origin rpy="0.0 0.0 0.0" xyz=" 0.0 0.0 0.1206"/>
+    <parent link="link4"/>
+    <child link="flange"/>
+  </joint>
 </robot>
