Commit message: Gazebo improvements

File: src/AR3/urdf/AR3.urdf (robot description, URDF)
Before this commit: robot AR3_Pedestal, 8 links, 7 joints
Links:
- removed link world
- link base: mass 1 -> 1.5
- link link1: mass 1 -> 1.5
- link link2: mass 1 -> 1.5
- link link3: mass 1 -> 1.5
- link link4: mass 1 -> 1.5
- link link5: mass 1 -> 1.5
- link link6: mass 1 -> 1.5
Joints:
- removed joint BaseJoint
- joint joint1: limit (none) -> lower=-1.57079632679 upper=1.57079632679 effort=30.0 velocity=10.0
- joint joint2: limit (none) -> lower=-1.57079632679 upper=3.14159265359 effort=30.0 velocity=10.0; origin xyz=0.06136563 -0.06786547 0.1390754 rpy=0 0 0 -> xyz=0.0508 -0.06786547 0.1390754 rpy=0 0 0
- joint joint3: limit (none) -> lower=-1.57079632679 upper=1.57079632679 effort=30.0 velocity=10.0; origin xyz=-0.015 0 0.305 rpy=0 0 0 -> xyz=-0.015 0 0.305 rpy=-1.57079632679 0 0
- joint joint4: limit (none) -> lower=-1.57079632679 upper=1.57079632679 effort=30.0 velocity=10.0; origin xyz=-0.0235 -0.0503 0 rpy=0 0 0 -> xyz=-0.038 -0.0503 0 rpy=0 0 0
- joint joint5: limit (none) -> lower=-1.57079632679 upper=1.57079632679 effort=30.0 velocity=10.0

File: src/AR3/urdf/AR3.xacro (robot description, xacro)
@@ -4,10 +4,10 @@
   <!-- Constants for robot dimensions -->
   <xacro:property name="PI" value="3.1415926535897931"/>
-  <xacro:property name="mass" value="1.5" /> <!-- arbitrary value for mass -->
-  <xacro:property name="width" value="0.1" /> <!-- Square dimensions (widthxwidth) of beams -->
-  <xacro:property name="height1" value=".1397" /> <!-- Link 1 -->
-  <xacro:property name="height2" value="0.306" /> <!-- Link 2 -->
-  <xacro:property name="height3" value="0.227" /> <!-- Link 3 -->
-  <xacro:property name="height4" value="0.1" /> <!-- Link 0 -->
+  <xacro:property name="mass" value="1.5" />
+  <xacro:property name="width" value="0.1" />
+  <xacro:property name="height1" value=".1397" />
+  <xacro:property name="height2" value="0.306" />
+  <xacro:property name="height3" value="0.227" />
+  <xacro:property name="height4" value="0.1" />
   <!-- Joint offsets -->
   <xacro:property name="joint1_x" value="0"/>

File: src/AR3/urdf/AR3_Pedestal.xacro (robot description, xacro)
@@ -2,9 +2,11 @@
 <!-- Revolute-Revolute Manipulator -->
 <robot name="AR3_Pedestal" xmlns:xacro="http://www.ros.org/wiki/xacro">
+  <!-- Import all Gazebo-customization elements, including Gazebo colors -->
+  <xacro:include filename="$(find AR3)/urdf/AR3.xacro" />
   <!-- Constants for robot dimensions -->
   <xacro:property name="PI" value="3.1415926535897931"/>
   <xacro:property name="mass" value=".4" /> <!-- arbitrary value for mass -->
-  <xacro:property name="width" value="0.1" /> <!-- Square dimensions (widthxwidth) of beams -->
-  <xacro:property name="height1" value=".25" />
+  <xacro:property name="width" value="0.4" /> <!-- Square dimensions (widthxwidth) of beams -->
+  <xacro:property name="height1" value=".6" />
   <!-- Used for fixing robot to Gazebo 'base_link' -->
   <link name="world"/>
@@ -37,16 +39,14 @@
     <parent link="world"/>
     <child link="stand"/>
-    <origin xyz="0 0 ${height1/2}" rpy="0 0 0"/>
+    <origin xyz="0 0 0" rpy="0 0 0"/>
     <axis xyz="0 0 1"/>
     <dynamics damping="0.7"/>
     <!-- <limit lower="${-PI/2}" upper="${PI/2}" effort="30.0" velocity="10.0"/> -->
   </joint>
-  <!-- Import all Gazebo-customization elements, including Gazebo colors -->
-  <xacro:include filename="$(find AR3)/urdf/AR3.xacro" />
   <!-- Stand to Robot -->
  <joint name="Stand_to_Robot" type="fixed">
     <parent link="stand"/>
     <child link="base"/>
-    <origin xyz="0 0 ${height1/2}" rpy="0 0 0"/>
+    <origin xyz="0 -.04755873 ${height1 + .04975}" rpy="0 0 0"/>
     <axis xyz="0 0 1"/>
     <dynamics damping="0.7"/>
