Commit message: Joint 4 rewiring fix

File: src/AR3/urdf/AR3.xacro (robot description, xacro)
@@ -4,5 +4,5 @@
   <!-- Constants for robot dimensions -->
   <xacro:property name="PI" value="3.1415926535897931"/>
-  <xacro:property name="mass" value="1" /> <!-- arbitrary value for mass -->
+  <xacro:property name="mass" value="1.5" /> <!-- arbitrary value for mass -->
   <xacro:property name="width" value="0.1" /> <!-- Square dimensions (widthxwidth) of beams -->
   <xacro:property name="height1" value=".1397" /> <!-- Link 1 -->
@@ -98,5 +98,5 @@
     <axis xyz="0 0 1"/>
     <dynamics damping="0.7"/>
-    <!-- <limit lower="${-PI/2}" upper="${PI/2}" effort="30.0" velocity="10.0"/> -->
+    <limit lower="${-PI/2}" upper="${PI/2}" effort="30.0" velocity="10.0"/>
   </joint>
   <!-- Link 2 -->
@@ -132,5 +132,5 @@
     <axis xyz="1 0 0"/>
     <dynamics damping="0.7"/>
-    <!-- <limit lower="${-PI/2}" upper="${PI/2}" effort="30.0" velocity="10.0"/> -->
+    <limit lower="${-PI/2}" upper="${PI}" effort="30.0" velocity="10.0"/>
   </joint>
   <!-- Link 3 -->
@@ -165,5 +165,5 @@
     <axis xyz="1 0 0"/>
     <dynamics damping="0.7"/>
-    <!-- <limit lower="${-PI/2}" upper="${PI/2}" effort="30.0" velocity="10.0"/> -->
+    <limit lower="${-PI/2}" upper="${PI/2}" effort="30.0" velocity="10.0"/>
   </joint>
   <!-- LINK 4-->
@@ -198,5 +198,5 @@
     <axis xyz="0 1 0"/>
     <dynamics damping="0.7"/>
-    <!-- <limit lower="${-PI/2}" upper="${PI/2}" effort="30.0" velocity="10.0"/> -->
+    <limit lower="${-PI/2}" upper="${PI/2}" effort="30.0" velocity="10.0"/>
   </joint>
   <!-- LINK 5-->
@@ -231,4 +231,5 @@
     <axis xyz="1 0 0"/>
     <dynamics damping="0.7"/>
+    <limit lower="${-PI/2}" upper="${PI/2}" effort="30.0" velocity="10.0"/>
   </joint>
   <!-- LINK 6-->

Commit message: Fixed URDF joint 3 rotation

File: src/AR3/urdf/AR3.xacro (robot description, xacro)
@@ -162,5 +162,5 @@
     <parent link="link2"/>
     <child link="link3"/>
-    <origin xyz="${joint3_x} ${joint3_y} ${joint3_z}" rpy="0 0 0"/>
+    <origin xyz="${joint3_x} ${joint3_y} ${joint3_z}" rpy="${-PI/2} 0 0"/>
     <axis xyz="1 0 0"/>
     <dynamics damping="0.7"/>

Commit message: Simulation and robot_controlelr improvements

File: src/AR3/urdf/AR3.xacro (robot description, xacro)
@@ -14,5 +14,5 @@
   <xacro:property name="joint1_y" value="0"/>
   <xacro:property name="joint1_z" value="0"/>
-  <xacro:property name="joint2_x" value=".06136563"/>
+  <xacro:property name="joint2_x" value=".0508"/>
   <xacro:property name="joint2_y" value="-.06786547"/>
   <xacro:property name="joint2_z" value=".13907540"/>
@@ -20,5 +20,5 @@
   <xacro:property name="joint3_y" value="0"/>
   <xacro:property name="joint3_z" value=".305"/>
-  <xacro:property name="joint4_x" value="-.0235"/>
+  <xacro:property name="joint4_x" value="-.038"/>
   <xacro:property name="joint4_y" value="-.0503"/>
   <xacro:property name="joint4_z" value="0"/>

Commit message: Replay working

File: src/AR3/urdf/AR3.xacro (robot description, xacro)
@@ -4,8 +4,8 @@
   <!-- Constants for robot dimensions -->
   <xacro:property name="PI" value="3.1415926535897931"/>
-  <xacro:property name="mass" value="1.5" />
+  <xacro:property name="mass" value="1.2" />
   <xacro:property name="width" value="0.1" />
   <xacro:property name="height1" value=".1397" />
-  <xacro:property name="height2" value="0.306" />
+  <xacro:property name="height2" value="0.206" />
   <xacro:property name="height3" value="0.227" />
   <xacro:property name="height4" value="0.1" />
