Commit message: Arduino tweaks

File: src/AR3/urdf/AR3_Pedestal.xacro (robot description, xacro)
@@ -28,5 +28,5 @@
       <inertial>
         <origin xyz="0 0 ${height1/2}" rpy="0 0 0"/>
-        <mass value="${mass}"/>
+        <mass value="200"/>
         <inertia
           ixx="${mass / 12.0 * (width*width + height1*height1)}" ixy="0.0" ixz="0.0"

Commit message: Edge angle and urdf improvements

File: src/AR3/urdf/AR3_Pedestal.xacro (robot description, xacro)
@@ -48,5 +48,5 @@
     <parent link="stand"/>
     <child link="base"/>
-    <origin xyz="0 -.04755873 ${height1 + .04975}" rpy="0 0 0"/>
+    <origin xyz="0 .04755873 ${height1 + .04975}" rpy="0 0 3.14159"/>
     <axis xyz="0 0 1"/>
     <dynamics damping="0.7"/>
