Commit message: base joint direction fix

File: src/AR3/urdf/AR3_Shelving.xacro (robot description, xacro)
@@ -80,5 +80,5 @@
     <parent link="world"/>
     <child link="shelving"/>
-    <origin xyz="0 .25 0" rpy="0 0 3.14"/>
+    <origin xyz=".1 .25 0" rpy="0 0 3.14"/>
     <axis xyz="0 0 1"/>
     <dynamics damping="0.7"/>
